File: AL_Controller.sch (KiCad schematic (older format))
At the start: 5 parts, among them U21 74181, U22 74181, U23 74AHC1G08, U24 a, U25 OctalBuffer

Commit message: Respin Counter
Parts:
- U23, U24: symbol 74xGxx:74AHC1G08 -> MAX7000CPU-Gen2-rescue:74AHC1G08-74xGxx
Changed lines of the file:
@@
 	2300 2250 2750 2250
 $Comp
-L 74xGxx:74AHC1G08 U23
+L MAX7000CPU-Gen2-rescue:74AHC1G08-74xGxx U23
 U 1 1 6101A286
 P 2750 2650
@@
 	2300 3300 2600 3300
 $Comp
-L 74xGxx:74AHC1G08 U24
+L MAX7000CPU-Gen2-rescue:74AHC1G08-74xGxx U24
 U 1 1 61022A3F
 P 2900 3250
