File: AL_Controller.sch (KiCad schematic (older format))
At the start: 5 parts, among them U21 74181, U22 74181, U23 74AHC1G08, U24 a, U25 OctalBuffer

Commit message: Stack Implementation
Parts:
- renumbered U21 to UI21, U22 to UI22, U25 to UI25
Connections:
- new net: UI21.~ (S3), UI25.~ (Out7) (x4)
- new net: UI22.~ (S3), UI25.~ (Out7) (x4)
- no-connect marks 0 -> 1
Changed lines of the file:
@@
 Ins3
 $Comp
-L CPU_internal_elements:OctalBuffer U25
+L CPU_internal_elements:OctalBuffer UI25
 U 1 1 610132D8
 P 3050 1300
-F 0 "U25" H 3050 1275 50  0000 C CNN
+F 0 "UI25" H 3050 1275 50  0000 C CNN
 F 1 "OctalBuffer" H 3050 1184 50  0000 C CNN
 F 2 "" H 3050 1300 50  0001 C CNN
@@
 U 1 1 6101A286
 P 2750 2650
-F 0 "U23" V 2725 2520 50  0000 R CNN
+AR Path="/6101A286" Ref="U23"  Part="1"
+AR Path="/60FFC927/6101A286" Ref="UI23"  Part="1"
+F 0 "UI23" V 2725 2520 50  0000 R CNN
 F 1 "74AHC1G08" H 2725 2826 50  0001 C CNN
 F 2 "" H 2750 2650 50  0001 C CNN
@@
 U 1 1 61022A3F
 P 2900 3250
-F 0 "U24" H 3050 3150 50  0000 C CNN
+AR Path="/61022A3F" Ref="U24"  Part="1"
+AR Path="/60FFC927/61022A3F" Ref="UI24"  Part="1"
+F 0 "UI24" H 3050 3150 50  0000 C CNN
 F 1 "a" H 2950 3000 50  0001 C CNN
 F 2 "" H 2900 3250 50  0001 C CNN
@@
 B3
 $Comp
-L CPU_internal_elements:74181 U21
+L CPU_internal_elements:74181 UI21
 U 1 1 61026E63
 P 1250 700
-F 0 "U21" H 1525 725 50  0000 C CNN
+F 0 "UI21" H 1525 725 50  0000 C CNN
 F 1 "74181" H 1525 634 50  0000 C CNN
 F 2 "" H 1250 700 50  0001 C CNN
@@
 $EndComp
 $Comp
-L CPU_internal_elements:74181 U22
+L CPU_internal_elements:74181 UI22
 U 1 1 61029705
 P 1300 2250
-F 0 "U22" H 1575 2275 50  0000 C CNN
+F 0 "UI22" H 1575 2275 50  0000 C CNN
 F 1 "74181" H 1575 2184 50  0000 C CNN
 F 2 "" H 1300 2250 50  0001 C CNN
@@
 Text Label 3350 2250 0    50   ~ 0
 O7
+NoConn ~ -17700 -11900
 $EndSCHEMATC

Commit message: Counter Layout
Parts:
- renumbered UI21 to UI1, UI25 to UI2, UI22 to UI3, U23 to UI4, U24 to UI5
Connections:
- new net: UI1.~ (S3), UI2.~ (Out7) (x4)
- new net: UI2.~ (Out7), UI3.~ (S3) (x4)
Changed lines of the file:
@@
 Ins3
 $Comp
-L CPU_internal_elements:OctalBuffer UI25
+L CPU_internal_elements:OctalBuffer UI2
 U 1 1 610132D8
 P 3050 1300
-F 0 "UI25" H 3050 1275 50  0000 C CNN
+F 0 "UI2" H 3050 1275 50  0000 C CNN
 F 1 "OctalBuffer" H 3050 1184 50  0000 C CNN
 F 2 "" H 3050 1300 50  0001 C CNN
@@
 	2300 2250 2750 2250
 $Comp
-L MAX7000CPU-Gen2-rescue:74AHC1G08-74xGxx U23
+L MAX7000CPU-Gen2-rescue:74AHC1G08-74xGxx UI?
 U 1 1 6101A286
 P 2750 2650
-AR Path="/6101A286" Ref="U23"  Part="1"
-AR Path="/60FFC927/6101A286" Ref="UI23"  Part="1"
-F 0 "UI23" V 2725 2520 50  0000 R CNN
+AR Path="/6101A286" Ref="UI?"  Part="1"
+AR Path="/60FFC927/6101A286" Ref="UI4"  Part="1"
+F 0 "UI4" V 2725 2520 50  0000 R CNN
 F 1 "74AHC1G08" H 2725 2826 50  0001 C CNN
 F 2 "" H 2750 2650 50  0001 C CNN
@@
 	2300 3300 2600 3300
 $Comp
-L MAX7000CPU-Gen2-rescue:74AHC1G08-74xGxx U24
+L MAX7000CPU-Gen2-rescue:74AHC1G08-74xGxx UI?
 U 1 1 61022A3F
 P 2900 3250
-AR Path="/61022A3F" Ref="U24"  Part="1"
-AR Path="/60FFC927/61022A3F" Ref="UI24"  Part="1"
-F 0 "UI24" H 3050 3150 50  0000 C CNN
+AR Path="/61022A3F" Ref="UI?"  Part="1"
+AR Path="/60FFC927/61022A3F" Ref="UI5"  Part="1"
+F 0 "UI5" H 3050 3150 50  0000 C CNN
 F 1 "a" H 2950 3000 50  0001 C CNN
 F 2 "" H 2900 3250 50  0001 C CNN
@@
 B3
 $Comp
-L CPU_internal_elements:74181 UI21
+L CPU_internal_elements:74181 UI1
 U 1 1 61026E63
 P 1250 700
-F 0 "UI21" H 1525 725 50  0000 C CNN
+F 0 "UI1" H 1525 725 50  0000 C CNN
 F 1 "74181" H 1525 634 50  0000 C CNN
 F 2 "" H 1250 700 50  0001 C CNN
@@
 $EndComp
 $Comp
-L CPU_internal_elements:74181 UI22
+L CPU_internal_elements:74181 UI3
 U 1 1 61029705
 P 1300 2250
-F 0 "UI22" H 1575 2275 50  0000 C CNN
+F 0 "UI3" H 1575 2275 50  0000 C CNN
 F 1 "74181" H 1575 2184 50  0000 C CNN
 F 2 "" H 1300 2250 50  0001 C CNN

Commit message: ksim production
Parts:
- added UI? (x3): 4013, symbol 4xxx:4013
- added UI? (x5): 4081, symbol 4xxx:4081
Connections:
- new net: UI1.~ (S3), UI2.~ (Out7) (x4)
- new net: UI2.~ (Out7), UI3.~ (S3) (x4)
- new net: UI?.1 (Q), UI?.2, UI?.5 (D) (x2)
- new net: UI?.2, UI?.2, UI?.2 (~Q)
- new net: UI?.1, UI?.1, UI?.1, UI?.2 (~Q), UI?.5 (D)
- new net: UI?.2, UI?.2 (~Q)
- new net: UI?.1, UI?.1, UI?.1 (Q)
- new net Count++: UI?.3
- new net Counter_Out: UI?.3
- new net Cycle_Reset: UI?.4 (R), UI?.4 (R), UI?.4 (R)
- new net GlobalClock: UI?.3 (C), UI?.3 (C), UI?.3 (C)
- new net Instruction_Read: UI?.3
- new net Module_Read: UI?.3
- new net RamAddr_DriveBus: UI?.3
- no-connect marks 1 -> 4
Changed lines of the file:
@@
 EELAYER 30 0
 EELAYER END
-$Descr A4 11693 8268
+$Descr A3 16535 11693
 encoding utf-8
 Sheet 2 2
@@
 O7
 NoConn ~ -17700 -11900
+$Comp
+L 4xxx:4013 UI?
+U 1 1 612C16D4
+P 5200 1400
+F 0 "UI?" H 5200 1881 50  0000 C CNN
+F 1 "4013" H 5200 1790 50  0000 C CNN
+F 2 "" H 5200 1400 50  0001 C CNN
+F 3 "http://www.onsemi.com/pub/Collateral/MC14013B-D.PDF" H 5200 1400 50  0001 C CNN
+	1    5200 1400
+	1    0    0    -1
+$EndComp
+$Comp
+L 4xxx:4013 UI?
+U 1 1 612C652D
+P 6150 1400
+F 0 "UI?" H 6150 1881 50  0000 C CNN
+F 1 "4013" H 6150 1790 50  0000 C CNN
+F 2 "" H 6150 1400 50  0001 C CNN
+F 3 "http://www.onsemi.com/pub/Collateral/MC14013B-D.PDF" H 6150 1400 50  0001 C CNN
+	1    6150 1400
+	1    0    0    -1
+$EndComp
+$Comp
+L 4xxx:4013 UI?
+U 1 1 612CB7A3
+P 7050 1400
+F 0 "UI?" H 7050 1881 50  0000 C CNN
+F 1 "4013" H 7050 1790 50  0000 C CNN
+F 2 "" H 7050 1400 50  0001 C CNN
+F 3 "http://www.onsemi.com/pub/Collateral/MC14013B-D.PDF" H 7050 1400 50  0001 C CNN
+	1    7050 1400
+	1    0    0    -1
+$EndComp
+Wire Wire Line
+	4900 850  4900 1300
+Wire Wire Line
+	5500 1300 5600 1300
+Connection ~ 5600 1300
+Wire Wire Line
+	5600 1300 5850 1300
+Wire Wire Line
+	6450 1300 6600 1300
+Connection ~ 6600 1300
+Wire Wire Line
+	6600 1300 6750 1300
+Wire Wire Line
+	7350 1500 7500 1500
+Wire Wire Line
+	7500 1500 7500 850
+Wire Wire Line
+	7500 850  4900 850
+Wire Wire Line
+	7350 1300 7550 1300
+Wire Wire Line
+	5850 1400 5850 1750
+Wire Wire Line
+	5850 1750 4900 1750
+Wire Wire Line
+	4900 1750 4900 1550
+Wire Wire Line
+	5850 1750 6750 1750
+Wire Wire Line
+	6750 1750 6750 1400
+Connection ~ 5850 1750
+Wire Wire Line
+	7050 1700 6150 1700
+Connection ~ 5200 1700
+Wire Wire Line
+	5200 1700 4750 1700
+Connection ~ 6150 1700
+Wire Wire Line
+	6150 1700 5200 1700
+NoConn ~ 5200 1100
+NoConn ~ 6150 1100
+NoConn ~ 7050 1100
+Wire Wire Line
+	5500 1500 5700 1500
+Wire Wire Line
+	6450 1500 6700 1500
+Wire Wire Line
+	6700 1500 6700 1800
+Wire Wire Line
+	7500 1500 7650 1500
+Connection ~ 7500 1500
+Wire Wire Line
+	7550 1800 7300 1800
+Wire Wire Line
+	7550 1300 7550 1800
+Wire Wire Line
+	7650 1850 7400 1850
+Wire Wire Line
+	7650 1500 7650 1850
+Wire Wire Line
+	6700 1800 7200 1800
+Wire Wire Line
+	6600 1900 7100 1900
+Wire Wire Line
+	6600 1300 6600 1900
+Wire Wire Line
+	5700 1950 7000 1950
+Wire Wire Line
+	5700 1500 5700 1950
+Wire Wire Line
+	5600 2000 6900 2000
+Wire Wire Line
+	5600 1300 5600 2000
+Wire Wire Line
+	7400 1850 7400 2050
+Wire Wire Line
+	7000 1950 7000 2250
+Text Label 8450 2150 0    50   ~ 0
+Count++
+$Comp
+L 4xxx:4081 UI?
+U 1 1 61319D67
+P 8150 2150
+F 0 "UI?" H 8150 2475 50  0000 C CNN
+F 1 "4081" H 8150 2384 50  0000 C CNN
+F 2 "" H 8150 2150 50  0001 C CNN
+F 3 "http://www.intersil.com/content/dam/Intersil/documents/cd40/cd4073bms-81bms-82bms.pdf" H 8150 2150 50  0001 C CNN
+	1    8150 2150
+	1    0    0    -1
+$EndComp
+$Comp
+L 4xxx:4081 UI?
+U 1 1 6131DB9C
+P 8150 2700
+F 0 "UI?" H 8150 3025 50  0000 C CNN
+F 1 "4081" H 8150 2934 50  0000 C CNN
+F 2 "" H 8150 2700 50  0001 C CNN
+F 3 "http://www.intersil.com/content/dam/Intersil/documents/cd40/cd4073bms-81bms-82bms.pdf" H 8150 2700 50  0001 C CNN
+	1    8150 2700
+	1    0    0    -1
+$EndComp
+Text Label 8450 2700 0    50   ~ 0
+Counter_Out
+Wire Wire Line
+	7400 2050 7400 2600
+Wire Wire Line
+	7400 2600 7850 2600
+Connection ~ 7400 2050
+Wire Wire Line
+	6900 2800 7850 2800
+Wire Wire Line
+	6900 2000 6900 2800
+Text Label 4750 1700 2    50   ~ 0
+Cycle_Reset
+Wire Wire Line
+	4750 1550 4750 1500
+Wire Wire Line
+	4750 1550 4900 1550
+Connection ~ 4900 1550
+Wire Wire Line
+	4900 1550 4900 1400
+Text Label 4750 1500 2    50   ~ 0
+GlobalClock
+$Comp
+L 4xxx:4081 UI?
+U 1 1 61327B02
+P 8150 3250
+F 0 "UI?" H 8150 3575 50  0000 C CNN
+F 1 "4081" H 8150 3484 50  0000 C CNN
+F 2 "" H 8150 3250 50  0001 C CNN
+F 3 "http://www.intersil.com/content/dam/Intersil/documents/cd40/cd4073bms-81bms-82bms.pdf" H 8150 3250 50  0001 C CNN
+	1    8150 3250
+	1    0    0    -1
+$EndComp
+Wire Wire Line
+	7400 2600 7400 3150
+Wire Wire Line
+	7400 3150 7850 3150
+Connection ~ 7400 2600
+Wire Wire Line
+	7100 3350 7850 3350
+Wire Wire Line
+	7100 1900 7100 3350
+Text Label 8450 3250 0    50   ~ 0
+Instruction_Read
+$Comp
+L 4xxx:4081 UI?
+U 1 1 6132F143
+P 8150 3800
+F 0 "UI?" H 8150 4125 50  0000 C CNN
+F 1 "4081" H 8150 4034 50  0000 C CNN
+F 2 "" H 8150 3800 50  0001 C CNN
+F 3 "http://www.intersil.com/content/dam/Intersil/documents/cd40/cd4073bms-81bms-82bms.pdf" H 8150 3800 50  0001 C CNN
+	1    8150 3800
+	1    0    0    -1
+$EndComp
+Text Label 8450 3800 0    50   ~ 0
+RamAddr_DriveBus
+Wire Wire Line
+	7300 3700 7850 3700
+Wire Wire Line
+	7300 1800 7300 3700
+Wire Wire Line
+	7000 2250 7000 3900
+Wire Wire Line
+	7000 3900 7850 3900
+Connection ~ 7000 2250
+Wire Wire Line
+	7400 2050 7850 2050
+Wire Wire Line
+	7000 2250 7850 2250
+$Comp
+L 4xxx:4081 UI?
+U 1 1 6133BDAB
+P 8150 4350
+F 0 "UI?" H 8150 4675 50  0000 C CNN
+F 1 "4081" H 8150 4584 50  0000 C CNN
+F 2 "" H 8150 4350 50  0001 C CNN
+F 3 "http://www.intersil.com/content/dam/Intersil/documents/cd40/cd4073bms-81bms-82bms.pdf" H 8150 4350 50  0001 C CNN
+	1    8150 4350
+	1    0    0    -1
+$EndComp
+Wire Wire Line
+	7300 3700 7300 4250
+Wire Wire Line
+	7300 4250 7850 4250
+Connection ~ 7300 3700
+Wire Wire Line
+	7200 4450 7850 4450
+Wire Wire Line
+	7200 1800 7200 4450
+Text Label 8450 4350 0    50   ~ 0
+Module_Read
 $EndSCHEMATC

Commit message: controller timing
Parts:
- removed UI4: 74AHC1G08, symbol MAX7000CPU-Gen2-rescue:74AHC1G08-74xGxx
- added UI? (x3): 4013, symbol 4xxx:4013
- added UI? (x2): 4081, symbol 4xxx:4081
- added UI?: 4071, symbol 4xxx:4071
Connections:
- net CarryOut is gone; now on net Ins5: UI3.~ (S3)
- net O0 is gone; now on net Bus7: UI2.~ (Out7)
- net O1 is gone; now on net Bus7: UI2.~ (Out7)
- net O2 is gone; now on net Bus7: UI2.~ (Out7)
- net O3 is gone; now on net Bus7: UI2.~ (Out7)
- net O4 is gone; now on net Bus7: UI2.~ (Out7)
- net O5 is gone; now on net Bus7: UI2.~ (Out7)
- net O6 is gone; now on net Bus7: UI2.~ (Out7)
- net O7 is gone; now on net Bus7: UI2.~ (Out7)
- net Instruction_Read: now also UI?.3 (C), UI?.3 (C)
- net Bus7: now reaches UI2.~ (Out7)
- net AequalB_Out: no longer names the net of UI5.4
- net AequalB_Out: now also UI?.5 (D)
- new net: UI1.~ (S3), UI2.~ (Out7) (x4)
- new net: UI2.~ (Out7), UI3.~ (S3) (x4)
- new net: UI3.~ (S3), UI?.5 (D)
- new net: UI?.1, UI?.1 (Q)
- new net: UI?.1, UI?.2 (~Q), UI?.5 (D)
- new net: UI?.1, UI?.3
- new net: UI?.2, UI?.3
- new net A=B_Flag: UI?.1 (Q)
- new net Bus0: UI2.~ (Out7)
- new net Bus1: UI2.~ (Out7)
- new net Bus2: UI2.~ (Out7)
- new net Bus3: UI2.~ (Out7)
- new net Bus4: UI2.~ (Out7)
- new net Bus5: UI2.~ (Out7)
- new net Bus6: UI2.~ (Out7)
- new net CLK_Select: UI?.3 (C)
- new net CarryFlag: UI?.1 (Q)
- new net GlobalCLK: UI?.3
- new net SlowCLK: UI?.2
- new net UserCLK: UI?.2
- no-connect marks 4 -> 8
Other:
- moved on the sheet: UI5
Changed lines of the file:
@@
 Wire Wire Line
 	2300 2250 2750 2250
-$Comp
-L MAX7000CPU-Gen2-rescue:74AHC1G08-74xGxx UI?
-U 1 1 6101A286
-P 2750 2650
-AR Path="/6101A286" Ref="UI?"  Part="1"
-AR Path="/60FFC927/6101A286" Ref="UI4"  Part="1"
-F 0 "UI4" V 2725 2520 50  0000 R CNN
-F 1 "74AHC1G08" H 2725 2826 50  0001 C CNN
-F 2 "" H 2750 2650 50  0001 C CNN
-F 3 "http://www.ti.com/lit/sg/scyt129e/scyt129e.pdf" H 2750 2650 50  0001 C CNN
-	1    2750 2650
-	0    -1   -1   0
-$EndComp
-Text Label 2800 2950 3    50   ~ 0
-Ins6
-Text Label 2700 2950 3    50   ~ 0
-Ins7
 Wire Wire Line
 	2050 1500 2050 2450
@@
 	2350 2450 2350 3200
 Wire Wire Line
-	2350 3200 2600 3200
-Wire Wire Line
 	2100 3050 2300 3050
 Wire Wire Line
 	2300 3050 2300 3300
-Wire Wire Line
-	2300 3300 2600 3300
 $Comp
 L MAX7000CPU-Gen2-rescue:74AHC1G08-74xGxx UI?
 U 1 1 61022A3F
-P 2900 3250
+P 2650 3250
 AR Path="/61022A3F" Ref="UI?"  Part="1"
 AR Path="/60FFC927/61022A3F" Ref="UI5"  Part="1"
-F 0 "UI5" H 3050 3150 50  0000 C CNN
-F 1 "a" H 2950 3000 50  0001 C CNN
-F 2 "" H 2900 3250 50  0001 C CNN
-F 3 "http://www.ti.com/lit/sg/scyt129e/scyt129e.pdf" H 2900 3250 50  0001 C CNN
-	1    2900 3250
-	1    0    0    -1
-$EndComp
-Text Label 2100 2950 0    50   ~ 0
-CarryOut
-Text Label 3150 3250 0    50   ~ 0
-AequalB_Out
+F 0 "UI5" H 2800 3150 50  0000 C CNN
+F 1 "a" H 2700 3000 50  0001 C CNN
+F 2 "" H 2650 3250 50  0001 C CNN
+F 3 "http://www.ti.com/lit/sg/scyt129e/scyt129e.pdf" H 2650 3250 50  0001 C CNN
+	1    2650 3250
+	1    0    0    -1
+$EndComp
 Text Label 1000 900  2    50   ~ 0
 A0
@@
 Text Label 1050 3200 2    50   ~ 0
 B7
-Text Label 3350 1550 0    50   ~ 0
-O0
-Text Label 3350 1650 0    50   ~ 0
-O1
-Text Label 3350 1750 0    50   ~ 0
-O2
-Text Label 3350 1850 0    50   ~ 0
-O3
-Text Label 3350 1950 0    50   ~ 0
-O4
-Text Label 3350 2050 0    50   ~ 0
-O5
-Text Label 3350 2150 0    50   ~ 0
-O6
-Text Label 3350 2250 0    50   ~ 0
-O7
 NoConn ~ -17700 -11900
 $Comp
@@
 Text Label 8450 4350 0    50   ~ 0
 Module_Read
+$Comp
+L 4xxx:4013 UI?
+U 1 1 6132E2C1
+P 10250 1200
+F 0 "UI?" H 10250 1681 50  0000 C CNN
+F 1 "4013" H 10250 1590 50  0000 C CNN
+F 2 "" H 10250 1200 50  0001 C CNN
+F 3 "http://www.onsemi.com/pub/Collateral/MC14013B-D.PDF" H 10250 1200 50  0001 C CNN
+	1    10250 1200
+	1    0    0    -1
+$EndComp
+$Comp
+L 4xxx:4081 UI?
+U 1 1 61335FB0
+P 10350 2050
+F 0 "UI?" H 10350 2375 50  0000 C CNN
+F 1 "4081" H 10350 2284 50  0000 C CNN
+F 2 "" H 10350 2050 50  0001 C CNN
+F 3 "http://www.intersil.com/content/dam/Intersil/documents/cd40/cd4073bms-81bms-82bms.pdf" H 10350 2050 50  0001 C CNN
+	1    10350 2050
+	1    0    0    -1
+$EndComp
+Wire Wire Line
+	10550 1300 10550 1600
+Wire Wire Line
+	10550 1600 9900 1600
+Wire Wire Line
+	9900 1600 9900 1100
+Wire Wire Line
+	9900 1100 9950 1100
+Wire Wire Line
+	9950 1200 9650 1200
+Text Label 9650 1200 2    50   ~ 0
+CLK_Select
+$Comp
+L 4xxx:4081 UI?
+U 1 1 61344617
+P 10350 2600
+F 0 "UI?" H 10350 2925 50  0000 C CNN
+F 1 "4081" H 10350 2834 50  0000 C CNN
+F 2 "" H 10350 2600 50  0001 C CNN
+F 3 "http://www.intersil.com/content/dam/Intersil/documents/cd40/cd4073bms-81bms-82bms.pdf" H 10350 2600 50  0001 C CNN
+	1    10350 2600
+	1    0    0    -1
+$EndComp
+Wire Wire Line
+	9900 1600 9900 1950
+Wire Wire Line
+	9900 1950 10050 1950
+Connection ~ 9900 1600
+Wire Wire Line
+	10550 1100 10600 1100
+Wire Wire Line
+	10600 1100 10600 1650
+Wire Wire Line
+	10600 1650 9950 1650
+Wire Wire Line
+	9950 1650 9950 2500
+Wire Wire Line
+	9950 2500 10050 2500
+Wire Wire Line
+	10050 2150 9700 2150
+Wire Wire Line
+	10050 2700 9700 2700
+Text Label 9700 2150 2    50   ~ 0
+UserCLK
+Text Label 9700 2700 2    50   ~ 0
+SlowCLK
+$Comp
+L 4xxx:4071 UI?
+U 1 1 6135491E
+P 11200 2250
+F 0 "UI?" H 11200 2575 50  0000 C CNN
+F 1 "4071" H 11200 2484 50  0000 C CNN
+F 2 "" H 11200 2250 50  0001 C CNN
+F 3 "http://www.intersil.com/content/dam/Intersil/documents/cd40/cd4071bms-72bms-75bms.pdf" H 11200 2250 50  0001 C CNN
+	1    11200 2250
+	1    0    0    -1
+$EndComp
+Wire Wire Line
+	10650 2050 10650 2150
+Wire Wire Line
+	10650 2150 10900 2150
+Wire Wire Line
+	10650 2600 10650 2350
+Wire Wire Line
+	10650 2350 10900 2350
+Text Label 11500 2250 0    50   ~ 0
+GlobalCLK
+Text Label 3350 1550 0    50   ~ 0
+Bus0
+Text Label 3350 1650 0    50   ~ 0
+Bus1
+Text Label 3350 1750 0    50   ~ 0
+Bus2
+Text Label 3350 1850 0    50   ~ 0
+Bus3
+Text Label 3350 1950 0    50   ~ 0
+Bus4
+Text Label 3350 2050 0    50   ~ 0
+Bus5
+Text Label 3350 2150 0    50   ~ 0
+Bus6
+Text Label 3350 2250 0    50   ~ 0
+Bus7
+$Comp
+L 4xxx:4013 UI?
+U 1 1 613C0330
+P 3600 3000
+F 0 "UI?" H 3600 3481 50  0000 C CNN
+F 1 "4013" H 3600 3390 50  0000 C CNN
+F 2 "" H 3600 3000 50  0001 C CNN
+F 3 "http://www.onsemi.com/pub/Collateral/MC14013B-D.PDF" H 3600 3000 50  0001 C CNN
+	1    3600 3000
+	1    0    0    -1
+$EndComp
+Wire Wire Line
+	2300 3300 2350 3300
+Wire Wire Line
+	2100 2950 2800 2950
+Wire Wire Line
+	2800 2950 2800 2900
+Wire Wire Line
+	2800 2900 3300 2900
+$Comp
+L 4xxx:4013 UI?
+U 1 1 613ED860
+P 3600 3850
+F 0 "UI?" H 3600 4331 50  0000 C CNN
+F 1 "4013" H 3600 4240 50  0000 C CNN
+F 2 "" H 3600 3850 50  0001 C CNN
+F 3 "http://www.onsemi.com/pub/Collateral/MC14013B-D.PDF" H 3600 3850 50  0001 C CNN
+	1    3600 3850
+	1    0    0    -1
+$EndComp
+NoConn ~ 3600 3300
+NoConn ~ 3600 2700
+NoConn ~ 3600 3550
+NoConn ~ 3600 4150
+Wire Wire Line
+	2900 3250 3300 3250
+Wire Wire Line
+	3300 3250 3300 3750
+Wire Wire Line
+	3300 3000 3200 3000
+Wire Wire Line
+	3200 3000 3200 3550
+Wire Wire Line
+	3200 3850 3300 3850
+Text Label 2950 3550 2    50   ~ 0
+Instruction_Read
+Wire Wire Line
+	2950 3550 3200 3550
+Connection ~ 3200 3550
+Wire Wire Line
+	3200 3550 3200 3850
+Text Label 3900 2900 0    50   ~ 0
+CarryFlag
+Text Label 3900 3750 0    50   ~ 0
+A=B_Flag
 $EndSCHEMATC

Commit message: other changes
Parts:
- removed UI5: a, symbol MAX7000CPU-Gen2-rescue:74AHC1G08-74xGxx
- added UI? (x5): 4068, symbol 4xxx_IEEE:4068
- added UI? (x6): 4081, symbol 4xxx:4081
- added UI? (x8): 74LS04, symbol 74xx:74LS04
Connections:
- net labels added: ALU_Enable, ARead, BRead, Ins6, Ins7, JumpEnable
- wire segments 113 -> 259
- no-connect marks 8 -> 12

Commit message: chchchanges
Parts:
- added UI? (x9): 4068, symbol 4xxx_IEEE:4068
- added UI? (x6): 4081, symbol 4xxx:4081
Connections:
- net labels added: DSP_Read, High_Addr_Read, JumpBuffer_Read_High, JumpBuffer_Read_Low, Low_Addr_Read, MemWriteControl, MemoryOutput, StackCountDown, StackCountUp
- wire segments 259 -> 425
