File: MAX7000CPU-Gen2.sch (KiCad schematic (older format))
At the start: 98 parts, among them J1 Conn_02x05_Odd_Even, J2 Conn_01x08_Male, J3 Conn_01x08_Male, J4 Conn_01x08_Male, J5 Conn_01x08_Male, J6 Conn_01x08_Male, J7 Conn_01x05_Male, SW1 SW_Push, SW2 SW_Push, SW4 SW_Push, U1 NE555P, U13 74LS573, U14 74LS573, U15 74LS573, U16 74LS573, U17 EPM7128slc84-15n, U19 74LS241, U2 NE555P, U20 74LS241, U3 NE555P, U5 EPM7128slc84-15n, U6 74LS573, U7 SN74HC161N, U8 SN74HC161N

Commit message: Forked from GEN1
Parts:
- renumbered SW4 to SW3
Other:
- note added: "CLK MODULE"
- note removed: "Design Note: Programming will be done using the \nMax7000 memory controller's access \nto the right port on the IDT7132, with a \nJTAG sequence, as a result of this addr\n11111111 in the instruction memory \ncannot be programed."
- moved on the sheet: C1, C2, C3, C4, C5, C6, R1, R2, R3, R4, R5, R6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

Commit message: Implementation
Parts:
- removed J3: Conn_01x08_Male, Connector_PinHeader_2.54mm:PinHeader_1x08_P2.54mm_Vertical, symbol Connector:Conn_01x08_Male
- added U? (x2): 74LS241, symbol 74xx:74LS241
- added U? (x2): SN74HC161N, Package_DIP:DIP-16_W7.62mm, symbol CPU_ics:SN74HC161N
- added U? (x4): 74LS574, Package_DIP:DIP-20_W7.62mm, symbol 74xx:74LS573
- added U?: AS6C1008-55PCN, DIP254P1524X393-32, symbol CPU_ics:AS6C1008-55PCN
- U13, U14, U15, U16, U6: value 74LS573 -> 74LS574
Connections:
- net +5V: now also U?.10 (ENT), U?.10 (ENT), U?.16 (VCC), U?.16 (VCC), U?.20 (VCC), U?.20 (VCC), U?.20 (VCC), U?.20 (VCC), U?.20 (VCC), U?.20 (VCC), U?.30 (CE2), U?.32 (VCC), U?.7 (ENP), U?.7 (ENP); no longer U19.1 (OEa), U19.19 (OEb), U20.1 (OEa), U20.19 (OEb)
- net A=B_FlagIn: no longer U5.15 (I/O)
- net A=B_Out: now also U5.75 (I/O); no longer U5.16 (I/O)
- net B0: now also J4.1 (Pin_1), R12.1, U13.19 (Q0), U13.2 (D0), U14.2 (D0), U15.2 (D0), U20.2 (I0a), U5.44 (I/O), U6.2 (D0), U?.13 (DQ0), U?.2 (D0), U?.2 (D0), U?.2 (D0), U?.2 (D0); no longer U15.19 (Q0), U5.67 (I/O)
- net B1: now also J4.2 (Pin_2), R13.1, U13.18 (Q1), U13.3 (D1), U14.3 (D1), U15.3 (D1), U20.4 (I1a), U5.45 (I/O), U6.3 (D1), U?.14 (DQ1), U?.3 (D1), U?.3 (D1), U?.3 (D1), U?.3 (D1); no longer U15.18 (Q1), U5.68 (I/O)
- net B2: now also J4.3 (Pin_3), R14.1, U13.17 (Q2), U13.4 (D2), U14.4 (D2), U15.4 (D2), U20.6 (I2a), U5.46 (I/O), U6.4 (D2), U?.15 (DQ2), U?.4 (D2), U?.4 (D2), U?.4 (D2), U?.4 (D2); no longer U15.17 (Q2), U5.69 (I/O)
- net B3: now also J4.4 (Pin_4), R15.1, U13.16 (Q3), U13.5 (D3), U14.5 (D3), U15.5 (D3), U20.8 (I3a), U5.48 (I/O), U6.5 (D3), U?.17 (DQ3), U?.5 (D3), U?.5 (D3), U?.5 (D3), U?.5 (D3); no longer U15.16 (Q3), U5.70 (I/O)
- net B4: now also J4.5 (Pin_5), R16.1, U13.15 (Q4), U13.6 (D4), U14.6 (D4), U15.6 (D4), U20.11 (I0b), U5.49 (I/O), U6.6 (D4), U?.18 (DQ4), U?.6 (D4), U?.6 (D4), U?.6 (D4), U?.6 (D4); no longer U15.15 (Q4), U5.73 (I/O)
- net B5: now also J4.6 (Pin_6), R17.1, U13.14 (Q5), U13.7 (D5), U14.7 (D5), U15.7 (D5), U20.13 (I1b), U5.50 (I/O), U6.7 (D5), U?.19 (DQ5), U?.7 (D5), U?.7 (D5), U?.7 (D5), U?.7 (D5); no longer U15.14 (Q5), U5.74 (I/O)
- net B6: now also J4.7 (Pin_7), R18.1, U13.13 (Q6), U13.8 (D6), U14.8 (D6), U15.8 (D6), U20.15 (I2b), U5.51 (I/O), U6.8 (D6), U?.20 (DQ6), U?.8 (D6), U?.8 (D6), U?.8 (D6), U?.8 (D6); no longer U15.13 (Q6), U5.76 (I/O)
- net B7: now also J4.8 (Pin_8), R19.1, U13.12 (Q7), U13.9 (D7), U14.9 (D7), U15.9 (D7), U20.17 (I3b), U5.52 (I/O), U6.9 (D7), U?.21 (DQ7), U?.9 (D7), U?.9 (D7), U?.9 (D7), U?.9 (D7); no longer U15.12 (Q7), U5.75 (I/O)
- net CLK: no longer U13.11 (Load), U17.4 (I/O), U5.51 (I/O), U7.2 (CLK)
- net CLK_Select: now also U5.20 (I/O); no longer U5.35 (I/O)
- net CarryFlagIn: no longer U5.11 (I/O)
- net CarryOut: now also U5.76 (I/O); no longer U5.12 (I/O)
- net CounterReset: now also U5.16 (I/O), U8.15 (RCO), U?.1 (*CLR), U?.1 (*CLR), U?.2 (CLK); no longer U17.46 (I/O)
- net Flag0In: no longer U5.17 (I/O)
- net Flag0Out: no longer U5.18 (I/O)
- net Flag1In: no longer U5.21 (I/O)
- net Flag1Out: no longer U5.20 (I/O)
- net Flag2In: no longer U5.25 (I/O)
- net Flag2Out: no longer U5.22 (I/O)
- net Flag3In: no longer U5.27 (I/O)
- net Flag3Out: no longer U5.24 (I/O)
- net Flag4In: no longer U5.29 (I/O)
- net Flag4Out: no longer U5.28 (I/O)
- net Flag5In: no longer U5.31 (I/O)
- net Flag5Out: no longer U5.30 (I/O)
- net FlagCLK: now also U5.77 (I/O); no longer U5.34 (I/O)
- net GND: now also U14.1 (OE), U15.1 (OE), U16.1 (OE), U19.1 (OEa), U19.19 (OEb), U20.1 (OEa), U20.19 (OEb), U6.1 (OE), U?.1 (OE), U?.1 (OE), U?.10 (GND), U?.10 (GND), U?.10 (GND), U?.10 (GND), U?.10 (GND), U?.10 (GND), U?.16 (VSS), U?.2 (A16), U?.22 (~CE), U?.8 (GND), U?.8 (GND)
- net Ins0: now also U5.4 (I/O), U?.19 (Q0); no longer U17.17 (I/O), U5.49 (I/O)
- net Ins1: now also U5.5 (I/O), U?.18 (Q1); no longer U17.15 (I/O), U5.48 (I/O)
- net Ins2: now also U5.6 (I/O), U?.17 (Q2); no longer U17.10 (I/O), U5.45 (I/O)
- net Ins3: now also U5.8 (I/O), U?.16 (Q3); no longer U17.11 (I/O), U5.46 (I/O)
- net Ins4: now also U5.9 (I/O), U?.15 (Q4); no longer U17.9 (I/O), U5.44 (I/O)
- net Ins5: now also U5.10 (I/O), U?.14 (Q5); no longer U17.8 (I/O), U5.41 (I/O)
- net Ins6: now also U5.11 (I/O), U?.13 (Q6); no longer U17.6 (I/O), U5.39 (I/O)
- net Ins7: now also U5.12 (I/O), U?.12 (Q7); no longer U17.5 (I/O), U5.40 (I/O)
- net JumpEnable: now also U5.31 (I/O), U?.9 (*LOAD), U?.9 (*LOAD); no longer U5.64 (I/O)
- net MemWriteControl: now also U5.35 (I/O), U?.29 (~WE); no longer U17.16 (I/O)
- net Qi0: no longer U17.58 (I/O)
- net Qi1: no longer U17.60 (I/O)
- net Qi2: no longer U17.61 (I/O)
- net Qi3: no longer U17.63 (I/O)
- net Qi4: no longer U17.64 (I/O)
- net Qi5: no longer U17.65 (I/O)
- net Qi6: no longer U17.67 (I/O)
- net Qi7: no longer U17.68 (I/O)
- net Qo0: no longer U17.70 (I/O)
- net Qo1: no longer U17.69 (I/O)
- net Qo2: no longer U17.74 (I/O)
- net Qo3: no longer U17.73 (I/O)
- net Qo4: no longer U17.75 (I/O)
- net Qo5: no longer U17.76 (I/O)
- net Qo6: no longer U17.77 (I/O)
- net Qo7: no longer U17.80 (I/O)
- net RegAControl: now also U5.25 (I/O); no longer U5.10 (I/O)
- net RegBControl: now also U5.27 (I/O); no longer U5.77 (I/O)
- net Reset: now also U5.15 (I/O); no longer U17.48 (I/O)
- net SlowCLK: now also U5.18 (I/O); no longer U5.33 (I/O)
- net UserCLK: now also U5.17 (I/O); no longer U5.36 (I/O)
- net MainRegOutputControl: now reaches U13.1 (OE)
- net MainRegOutputControl: now also U5.33 (I/O)
- net A0: no longer names the net of U5.79 (I/O)
- net A0: no longer U14.19 (Q0)
- net A1: no longer names the net of U5.80 (I/O)
- net A1: no longer U14.18 (Q1)
- net A2: no longer names the net of U5.81 (I/O)
- net A2: no longer U14.17 (Q2)
- net A3 renamed rA3
- net rA3: now also U5.57 (I/O); no longer U5.4 (I/O)
- net A4 renamed rA4
- net rA4: now also U5.58 (I/O); no longer U5.5 (I/O)
- net A5 renamed rA5
- net rA5: now also U5.60 (I/O); no longer U5.8 (I/O)
- net A6 renamed rA6
- net rA6: now also U5.61 (I/O); no longer U5.6 (I/O)
- net A7 renamed rA7
- net rA7: now also U5.63 (I/O); no longer U5.9 (I/O)
- net C0: no longer names the net of U7.14 (QA)
- net C0: now also U?.2 (I0a)
- net C1: no longer names the net of U7.13 (QB)
- net C1: now also U?.4 (I1a)
- net C2: no longer names the net of U7.12 (QC)
- net C2: now also U?.6 (I2a)
- net C3: no longer names the net of U7.11 (QD)
- net C3: now also U?.8 (I3a)
- net C4: no longer names the net of U8.14 (QA)
- net C4: now also U?.11 (I0b)
- net C5: no longer names the net of U8.13 (QB)
- net C5: now also U?.13 (I1b)
- net C6: no longer names the net of U8.12 (QC)
- net C6: now also U?.15 (I2b)
- net C7: no longer names the net of U8.11 (QD)
- net C7: now also U?.17 (I3b)
- net Comm0: no longer names the net of U17.81 (I/O)
- net Comm0: no longer U5.50 (I/O)
- net Comm1: no longer names the net of U17.79 (I/O)
- net Comm1: no longer U5.52 (I/O)
- net FastCLK: no longer names the net of U5.37 (I/O)
- removed net I0: U13.19 (Q0), U14.2 (D0), U15.2 (D0), U17.35 (I/O), U20.2 (I0a), U6.2 (D0)
- removed net I1: U13.18 (Q1), U14.3 (D1), U15.3 (D1), U17.39 (I/O), U20.4 (I1a), U6.3 (D1)
- removed net I2: U13.17 (Q2), U14.4 (D2), U15.4 (D2), U17.40 (I/O), U20.6 (I2a), U6.4 (D2)
- removed net I3: U13.16 (Q3), U14.5 (D3), U15.5 (D3), U17.36 (I/O), U20.8 (I3a), U6.5 (D3)
- removed net I4: U13.15 (Q4), U14.6 (D4), U15.6 (D4), U17.41 (I/O), U20.11 (I0b), U6.6 (D4)
- removed net I5: U13.14 (Q5), U14.7 (D5), U15.7 (D5), U17.44 (I/O), U20.13 (I1b), U6.7 (D5)
- removed net I6: U13.13 (Q6), U14.8 (D6), U15.8 (D6), U17.37 (I/O), U20.15 (I2b), U6.8 (D6)
- removed net I7: U13.12 (Q7), U14.9 (D7), U15.9 (D7), U17.45 (I/O), U20.17 (I3b), U6.9 (D7)
- net JumpRegLoad renamed LOWJumpRegLoad
- net LOWJumpRegLoad: now also U5.29 (I/O); no longer U5.65 (I/O)
- net M0: no longer names the net of U17.31 (I/O)
- net M1: no longer names the net of U17.20 (I/O)
- net M10: no longer names the net of U17.34 (I/O)
- net M2: no longer names the net of U17.29 (I/O)
- net M3: no longer names the net of U17.30 (I/O)
- net M4: no longer names the net of U17.22 (I/O)
- net M5: no longer names the net of U17.27 (I/O)
- net M6: no longer names the net of U17.28 (I/O)
- net M7: no longer names the net of U17.25 (I/O)
- net M8: no longer names the net of U17.24 (I/O)
- net M9: no longer names the net of U17.12 (I/O)
- net MemOutControl: no longer names the net of U17.18 (I/O)
- removed net O0: J4.1 (Pin_1), R12.1, U13.2 (D0), U17.57 (I/O), U5.54 (I/O)
- removed net O1: J4.2 (Pin_2), R13.1, U13.3 (D1), U17.56 (I/O), U5.55 (I/O)
- removed net O2: J4.3 (Pin_3), R14.1, U13.4 (D2), U17.55 (I/O), U5.56 (I/O)
- removed net O3: J4.4 (Pin_4), R15.1, U13.5 (D3), U17.52 (I/O), U5.57 (I/O)
- removed net O4: J4.5 (Pin_5), R16.1, U13.6 (D4), U17.51 (I/O), U5.58 (I/O)
- removed net O5: J4.6 (Pin_6), R17.1, U13.7 (D5), U17.54 (I/O), U5.60 (I/O)
- removed net O6: J4.7 (Pin_7), R18.1, U13.8 (D6), U17.50 (I/O), U5.61 (I/O)
- removed net O7: J4.8 (Pin_8), R19.1, U13.9 (D7), U17.49 (I/O), U5.63 (I/O)
- net RamAddrEnable: no longer names the net of U17.33 (I/O)
- net RamAddrLoad: no longer names the net of U17.21 (I/O)
- new net: U?.11 (QD), U?.8 (I3a)
- new net: U?.12 (QC), U?.6 (I2a)
- new net: U?.13 (QB), U?.4 (I1a)
- new net: U?.14 (QA), U?.2 (I0a)
- new net: U?.15 (RCO), U?.2 (CLK)
- new net: U?.19 (Q0), U?.3 (A)
- new net: U?.18 (Q1), U?.4 (B)
- new net: U?.17 (Q2), U?.5 (C)
- new net: U?.16 (Q3), U?.6 (D)
- new net: U?.11 (QD), U?.17 (I3b)
- new net: U?.12 (QC), U?.15 (I2b)
- new net: U?.13 (I1b), U?.13 (QB)
- new net: U?.11 (I0b), U?.14 (QA)
- new net: U?.15 (Q4), U?.3 (A)
- new net: U?.14 (Q5), U?.4 (B)
- new net: U?.13 (Q6), U?.5 (C)
- new net: U?.12 (Q7), U?.6 (D)
- new net Count: U5.21 (I/O), U7.2 (CLK)
- new net CounterOutControl: U5.22 (I/O), U?.1 (OEa), U?.1 (OEa), U?.19 (OEb), U?.19 (OEb)
- new net HIGHJumpRegLoad: U5.30 (I/O), U?.11 (Load)
- new net InsRegControl: U5.24 (I/O), U?.11 (Load)
- new net MainRegReadControl: U13.11 (Load), U5.28 (I/O)
- new net MemOutEnable: U5.34 (I/O), U?.24 (~OE)
- new net RAM_Addr_Enable: U?.1 (OE), U?.1 (OE)
- new net RAM_HighControl: U?.11 (Load)
- new net RAM_LowControl: U?.11 (Load)
- new net RA_H0: U?.18 (O0a), U?.19 (Q0), U?.27 (A8)
- new net RA_H1: U?.16 (O1a), U?.18 (Q1), U?.26 (A9)
- new net RA_H2: U?.14 (O2a), U?.17 (Q2), U?.23 (A10)
- new net RA_H3: U?.12 (O3a), U?.16 (Q3), U?.25 (A11)
- new net RA_H4: U?.15 (Q4), U?.4 (A12), U?.9 (O0b)
- new net RA_H5: U?.14 (Q5), U?.28 (A13), U?.7 (O1b)
- new net RA_H6: U?.13 (Q6), U?.3 (A14), U?.5 (O2b)
- new net RA_H7: U?.12 (Q7), U?.3 (O3b), U?.31 (A15)
- new net RA_L0: U?.12 (A0), U?.18 (O0a), U?.19 (Q0)
- new net RA_L1: U?.11 (A1), U?.16 (O1a), U?.18 (Q1)
- new net RA_L2: U?.10 (A2), U?.14 (O2a), U?.17 (Q2)
- new net RA_L3: U?.12 (O3a), U?.16 (Q3), U?.9 (A3)
- new net RA_L4: U?.15 (Q4), U?.8 (A4), U?.9 (O0b)
- new net RA_L5: U?.14 (Q5), U?.7 (A5), U?.7 (O1b)
- new net RA_L6: U?.13 (Q6), U?.5 (O2b), U?.6 (A6)
- new net RA_L7: U?.12 (Q7), U?.3 (O3b), U?.5 (A7)
- new net rA0: U14.19 (Q0), U5.54 (I/O)
- new net rA1: U14.18 (Q1), U5.55 (I/O)
- new net rA2: U14.17 (Q2), U5.56 (I/O)
- new net rB0: U15.19 (Q0), U5.64 (I/O)
- new net rB1: U15.18 (Q1), U5.65 (I/O)
- new net rB2: U15.17 (Q2), U5.67 (I/O)
- new net rB3: U15.16 (Q3), U5.68 (I/O)
- new net rB4: U15.15 (Q4), U5.69 (I/O)
- new net rB5: U15.14 (Q5), U5.70 (I/O)
- new net rB6: U15.13 (Q6), U5.73 (I/O)
- new net rB7: U15.12 (Q7), U5.74 (I/O)
- no-connect marks 14 -> 13
Other:
- note added: "Clock Module\n"
- note added: "Counter Module"
- note added: "General Purpose Registers"
- note added: "Interface"
- note added: "LEDs/drivers"
- note added: "Maybe Pull Chip enables to disable them when controllers arent running\n"
- note added: "RAM/Instructions"
- note removed: "CLK MODULE"
- note removed: "CRITICAL FLAW: THESE REGISTERS NEED TO BE TIED LOW NOT HIGH"
- moved on the sheet: C11, C12, C13, C14, C15, C16, C17, C18, C19, C20, C21, C22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

Commit message: CD4029 respin
Parts:
- added IC? (x8): CD4029BEE4, DIP794W53P254L1930H508Q16N, symbol CPU_ics:CD4029BEE4
- gave numbers to parts that had none: 9

Commit message: Respin Counter
Parts:
- removed IC? (x6): CD4029BEE4, DIP794W53P254L1930H508Q16N, symbol CPU_ics:CD4029BEE4
- removed U10, U7, U8, U9: SN74HC161N, Package_DIP:DIP-16_W7.62mm, symbol CPU_ics:SN74HC161N
- removed U12: 74LS241, symbol 74xx:74LS241
- removed U4: 74LS574, Package_DIP:DIP-20_W7.62mm, symbol 74xx:74LS573
- added U? (x3): CD4029BEE4, DIP794W53P254L1930H508Q16N, symbol CPU_ics:CD4029BEE4
- added U?: 74LS574, Package_DIP:DIP-20_W7.62mm, symbol MAX7000CPU-Gen2-rescue:74LS573-74xx
- added U?: 74LS241, symbol MAX7000CPU-Gen2-rescue:74LS241-74xx
- C1, C11, C12, C13, C14, C15, C16, C17, C18, C19, C2, C20, C21, C22, C23, C24, C25, C26, C27, C28, C29, C3, C30, C31, C32, C33, C34, C35, C36, C37, C38, C39, C4, C40, C41, C42, C5, C6: symbol Device:C -> MAX7000CPU-Gen2-rescue:C-Device
- D10, D11, D12, D13, D14, D15, D16, D17, D2, D3, D4, D5, D6, D7, D8, D9: symbol Device:LED -> MAX7000CPU-Gen2-rescue:LED-Device
- J1: symbol Connector_Generic:Conn_02x05_Odd_Even -> MAX7000CPU-Gen2-rescue:Conn_02x05_Odd_Even-Connector_Generic
- J2, J4, J5, J6: symbol Connector:Conn_01x08_Male -> MAX7000CPU-Gen2-rescue:Conn_01x08_Male-Connector
- J7: symbol Connector:Conn_01x05_Male -> MAX7000CPU-Gen2-rescue:Conn_01x05_Male-Connector
- R1, R12, R13, R14, R15, R16, R17, R18, R19, R2, R20, R21, R22, R23, R24, R3, R4, R5, R6: symbol Device:R -> MAX7000CPU-Gen2-rescue:R-Device
- RV1: symbol Device:R_POT -> MAX7000CPU-Gen2-rescue:R_POT-Device
- SW1, SW2, SW3: symbol Switch:SW_Push -> MAX7000CPU-Gen2-rescue:SW_Push-Switch
- U1, U2, U3: symbol Timer:NE555P -> MAX7000CPU-Gen2-rescue:NE555P-Timer
- U11, U19, U20: symbol 74xx:74LS241 -> MAX7000CPU-Gen2-rescue:74LS241-74xx
- U13, U14, U15, U16, U18, U26, U28, U6: symbol 74xx:74LS573 -> MAX7000CPU-Gen2-rescue:74LS573-74xx
- gave numbers to parts that had none: 1
Connections:
- net +5V: now also U?.10 (UP/DOWN), U?.16 (VDD), U?.9 (BINARY/DECADE), U?.10 (UP/DOWN), U?.10 (UP/DOWN), U?.10 (UP/DOWN), U?.16 (VDD), U?.16 (VDD), U?.16 (VDD), U?.20 (VCC), U?.20 (VCC), U?.9 (BINARY/DECADE), U?.9 (BINARY/DECADE), U?.9 (BINARY/DECADE)
- net B0: now also U?.2 (D0)
- net B1: now also U?.3 (D1)
- net B2: now also U?.4 (D2)
- net B3: now also U?.5 (D3)
- net B4: now also U?.6 (D4)
- net B5: now also U?.7 (D5)
- net B6: now also U?.8 (D6)
- net B7: now also U?.9 (D7)
- net Count: now also U?.15 (CLOCK), U?.15 (CLOCK), U?.15 (CLOCK), U?.15 (CLOCK)
- net CounterOutControl: now also U?.1 (OEa), U?.19 (OEb)
- net GND: now also U?.5 (~CARRYIN), U?.8 (VSS), U?.1 (OE), U?.10 (GND), U?.10 (GND), U?.8 (VSS), U?.8 (VSS), U?.8 (VSS)
- net HIGHJumpRegLoad: now also U?.11 (Load)
- net JumpEnable: now also U?.1 (PRESET_ENABLE), U?.1 (PRESET_ENABLE), U?.1 (PRESET_ENABLE), U?.1 (PRESET_ENABLE)
- net RA_H0: now also U?.18 (O0a)
- net RA_H1: now also U?.16 (O1a)
- net RA_H2: now also U?.14 (O2a)
- net RA_H3: now also U?.12 (O3a)
- net RA_H4: now also U?.9 (O0b)
- net RA_H5: now also U?.7 (O1b)
- net RA_H6: now also U?.5 (O2b)
- net RA_H7: now also U?.3 (O3b)
- net at U11.8 (I3a): now also U?.2 (Q4)
- net at U11.6 (I2a): now also U?.14 (Q3)
- net at U11.4 (I1a): now also U?.11 (Q2)
- net at U11.2 (I0a): now also U?.6 (Q1)
- net at U6.19 (Q0): now also U?.4 (JAM1)
- net at U6.18 (Q1): now also U?.12 (JAM2)
- net at U6.17 (Q2): now also U?.13 (JAM3)
- net at U6.16 (Q3): now also U?.3 (JAM4)
- net at U11.17 (I3b): now also U?.2 (Q4)
- net at U11.15 (I2b): now also U?.14 (Q3)
- net at U11.13 (I1b): now also U?.11 (Q2)
- net at U11.11 (I0b): now also U?.6 (Q1)
- net at U6.15 (Q4): now also U?.4 (JAM1)
- net at U6.14 (Q5): now also U?.12 (JAM2)
- net at U6.13 (Q6): now also U?.13 (JAM3)
- net at U6.12 (Q7): now also U?.3 (JAM4)
- net at U?.7 (~CARRY_OUT): now also U?.5 (~CARRYIN)
- new net: U?.5 (~CARRYIN), U?.7 (~CARRY_OUT) (x2)
- new net: U?.12 (Q7), U?.3 (JAM4)
- new net: U?.13 (JAM3), U?.13 (Q6)
- new net: U?.12 (JAM2), U?.14 (Q5)
- new net: U?.15 (Q4), U?.4 (JAM1)
- new net: U?.16 (Q3), U?.3 (JAM4)
- new net: U?.13 (JAM3), U?.17 (Q2)
- new net: U?.12 (JAM2), U?.18 (Q1)
- new net: U?.19 (Q0), U?.4 (JAM1)
- new net: U?.11 (I0b), U?.6 (Q1)
- new net: U?.11 (Q2), U?.13 (I1b)
- new net: U?.14 (Q3), U?.15 (I2b)
- new net: U?.17 (I3b), U?.2 (Q4)
- new net: U?.2 (I0a), U?.6 (Q1)
- new net: U?.11 (Q2), U?.4 (I1a)
- new net: U?.14 (Q3), U?.6 (I2a)
- new net: U?.2 (Q4), U?.8 (I3a)
- no-connect marks 13 -> 12
Other:
- moved on the sheet: U6, U?

Commit message: Stack Implementation
Parts:
- removed J6: Conn_01x08_Male, Connector_PinHeader_2.54mm:PinHeader_1x08_P2.54mm_Vertical, symbol MAX7000CPU-Gen2-rescue:Conn_01x08_Male-Connector
- removed U16: 74LS574, Package_DIP:DIP-20_W7.62mm, symbol MAX7000CPU-Gen2-rescue:74LS573-74xx
- removed U17: EPM7128slc84-15n, Package_LCC:PLCC-84_THT-Socket, symbol CPU_ics:EPM7128slc84-15n
- removed U?: CD4029BEE4, DIP794W53P254L1930H508Q16N, symbol CPU_ics:CD4029BEE4
- added U21, U22, U23, U24: CD4029BEE4, DIP794W53P254L1930H508Q16N, symbol CPU_ics:CD4029BEE4
- added U25, U26: 74LS241, symbol MAX7000CPU-Gen2-rescue:74LS241-74xx
- added U28: 74LS574, Package_DIP:DIP-20_W7.62mm, symbol MAX7000CPU-Gen2-rescue:74LS573-74xx
- gave numbers to parts that had none: 6
- renumbered C39 to C10, C42 to C7, C41 to C8, C40 to C9, U11 to U13, U20 to U15, U19 to U16, U18 to U17, U26 to U18, U27 to U19, U28 to U20, U5 to U29, U13 to U4, U14 to U5, U15 to U6, U6 to U7
Connections:
- net CounterReset is gone; now on net UserCLK: U29.16 (I/O)
- net +5V: now also U21.16 (VDD), U21.9 (BINARY/DECADE), U22.16 (VDD), U22.9 (BINARY/DECADE), U23.16 (VDD), U23.9 (BINARY/DECADE), U24.16 (VDD), U24.9 (BINARY/DECADE), U25.20 (VCC), U26.20 (VCC), U28.20 (VCC)
- net B0: now also U21.4 (JAM1), U23.4 (JAM1), U28.2 (D0)
- net B1: now also U21.12 (JAM2), U23.12 (JAM2), U28.3 (D1)
- net B2: now also U21.13 (JAM3), U23.13 (JAM3), U28.4 (D2)
- net B3: now also U21.3 (JAM4), U23.3 (JAM4), U28.5 (D3)
- net B4: now also U22.4 (JAM1), U24.4 (JAM1), U28.6 (D4)
- net B5: now also U22.12 (JAM2), U24.12 (JAM2), U28.7 (D5)
- net B6: now also U22.13 (JAM3), U24.13 (JAM3), U28.8 (D6)
- net B7: now also U22.3 (JAM4), U24.3 (JAM4), U28.9 (D7)
- net CLK: now also U29.79 (I/O)
- net CLK_Select: now also U29.18 (I/O); no longer U29.20 (I/O)
- net Count: now also U29.20 (I/O); no longer U29.21 (I/O)
- net CounterOutControl: now also U29.21 (I/O); no longer U29.22 (I/O)
- net GND: now also U21.5 (~CARRYIN), U21.8 (VSS), U22.8 (VSS), U23.8 (VSS), U24.8 (VSS), U25.10 (GND), U26.10 (GND), U28.1 (OE), U28.10 (GND)
- net HIGHJumpRegLoad: now also U29.29 (I/O); no longer U29.30 (I/O)
- net InsRegControl: now also U29.22 (I/O); no longer U29.24 (I/O)
- net JumpEnable: now also U29.30 (I/O); no longer U29.31 (I/O)
- net LOWJumpRegLoad: now also U29.28 (I/O); no longer U29.29 (I/O)
- net MainRegOutputControl: now also U29.31 (I/O); no longer U29.33 (I/O)
- net MainRegReadControl: now also U29.27 (I/O); no longer U29.28 (I/O)
- net MemOutEnable: now also U29.33 (I/O); no longer U29.34 (I/O)
- net MemWriteControl: now also U29.34 (I/O); no longer U29.35 (I/O)
- net Qo0: now also U28.12 (Q7)
- net Qo1: now also U28.13 (Q6)
- net Qo2: now also U28.14 (Q5)
- net Qo3: now also U28.15 (Q4)
- net Qo4: now also U28.16 (Q3)
- net Qo5: now also U28.17 (Q2)
- net Qo6: now also U28.18 (Q1)
- net Qo7: now also U28.19 (Q0)
- net RAM_Addr_Enable: now also U29.37 (I/O)
- net RAM_HighControl: now also U29.36 (I/O)
- net RAM_LowControl: now also U29.35 (I/O)
- net RA_H0: now also U26.18 (O0a)
- net RA_H1: now also U26.16 (O1a)
- net RA_H2: now also U26.14 (O2a)
- net RA_H3: now also U26.12 (O3a)
- net RA_H4: now also U26.9 (O0b)
- net RA_H5: now also U26.7 (O1b)
- net RA_H6: now also U26.5 (O2b)
- net RA_H7: now also U26.3 (O3b)
- net RA_L0: now also U25.18 (O0a)
- net RA_L1: now also U25.16 (O1a)
- net RA_L2: now also U25.14 (O2a)
- net RA_L3: now also U25.12 (O3a)
- net RA_L4: now also U25.9 (O0b)
- net RA_L5: now also U25.7 (O1b)
- net RA_L6: now also U25.5 (O2b)
- net RA_L7: now also U25.3 (O3b)
- net RegAControl: now also U29.24 (I/O); no longer U29.25 (I/O)
- net RegBControl: now also U29.25 (I/O); no longer U29.27 (I/O)
- net SlowCLK: now also U29.17 (I/O); no longer U29.18 (I/O)
- net UserCLK: no longer U29.17 (I/O)
- net StackCount: now reaches U29.39 (I/O)
- net StackCount: now also U21.15 (CLOCK), U22.15 (CLOCK), U23.15 (CLOCK), U24.15 (CLOCK)
- net StackOutControl: now reaches U29.40 (I/O)
- net StackOutControl: now also U25.1 (OEa), U25.19 (OEb), U26.1 (OEa), U26.19 (OEb)
- net DSPcontrol: now reaches U29.41 (I/O)
- net DSPcontrol: now also U28.11 (Load)
- net SYNC: now reaches U29.80 (I/O)
- net SYNC: now also J7.2 (Pin_2)
- net STATE: now reaches U29.81 (I/O)
- net STATE: now also J7.3 (Pin_3)
- net A=B_Out renamed LowStackJump
- net LowStackJump: now also U21.1 (PRESET_ENABLE), U22.1 (PRESET_ENABLE); no longer J7.3 (Pin_3)
- net CarryOut renamed HighStackJump
- net HighStackJump: now also U23.1 (PRESET_ENABLE), U24.1 (PRESET_ENABLE); no longer J7.2 (Pin_2)
- net FlagCLK renamed StackCountDirection
- net StackCountDirection: now also U21.10 (UP/DOWN), U22.10 (UP/DOWN), U23.10 (UP/DOWN), U24.10 (UP/DOWN)
- new net: U22.6 (Q1), U25.11 (I0b)
- new net: U22.11 (Q2), U25.13 (I1b)
- new net: U22.14 (Q3), U25.15 (I2b)
- new net: U22.2 (Q4), U25.17 (I3b)
- new net: U21.6 (Q1), U25.2 (I0a)
- new net: U21.11 (Q2), U25.4 (I1a)
- new net: U21.14 (Q3), U25.6 (I2a)
- new net: U21.2 (Q4), U25.8 (I3a)
- new net: U21.7 (~CARRY_OUT), U22.5 (~CARRYIN)
- new net: U22.7 (~CARRY_OUT), U23.5 (~CARRYIN)
- new net: U24.6 (Q1), U26.11 (I0b)
- new net: U24.11 (Q2), U26.13 (I1b)
- new net: U24.14 (Q3), U26.15 (I2b)
- new net: U24.2 (Q4), U26.17 (I3b)
- new net: U23.6 (Q1), U26.2 (I0a)
- new net: U23.11 (Q2), U26.4 (I1a)
- new net: U23.14 (Q3), U26.6 (I2a)
- new net: U23.2 (Q4), U26.8 (I3a)
- new net: U23.7 (~CARRY_OUT), U24.5 (~CARRYIN)
- no-connect marks 12 -> 10
Other:
- note added: "Decoupling"
- note added: "Flags are stored in control unit"
- note added: "Speciality Registers"
- note added: "Stack \nCounter"
- moved on the sheet: C10, C11, C12, C13, C14, C15, C16, C17, C18, C19, C20, C21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

Commit message: Footprint Association
Parts:
- U10, U11, U12, U21, U22, U23, U24, U9: footprint DIP794W53P254L1930H508Q16N -> Package_DIP:DIP-16_W7.62mm
- U13, U14, U25, U26: footprint (none) -> Package_DIP:DIP-20_W7.62mm
- U19: footprint DIP254P1524X393-32 -> Package_DIP:DIP-32_W15.24mm
Changed lines of the file:
@@
 F 0 "U13" H 4250 4300 50  0000 C CNN
 F 1 "74LS241" H 4350 4200 50  0000 C CNN
-F 2 "" H 4650 3550 50  0001 C CNN
+F 2 "Package_DIP:DIP-20_W7.62mm" H 4650 3550 50  0001 C CNN
 F 3 "http://www.ti.com/lit/ds/symlink/sn74ls241.pdf" H 4650 3550 50  0001 C CNN
 	1    4650 3550
@@
 F 0 "U19" H 3450 7665 50  0000 C CNN
 F 1 "AS6C1008-55PCN" H 3450 7574 50  0000 C CNN
-F 2 "DIP254P1524X393-32" H 3200 8350 50  0001 L CNN
+F 2 "Package_DIP:DIP-32_W15.24mm" H 3200 8350 50  0001 L CNN
 F 3 "http://componentsearchengine.com/Datasheets/1/AS6C1008-55PCN.pdf" H 3200 8250 50  0001 L CNN
 F 4 "CMOS SRAM" H 3200 8150 50  0001 L CNN "Description"
@@
 F 0 "U9" H 2450 3050 50  0000 C CNN
 F 1 "CD4029BEE4" H 2650 2950 50  0000 C CNN
-F 2 "DIP794W53P254L1930H508Q16N" H 4100 2950 50  0001 L CNN
+F 2 "Package_DIP:DIP-16_W7.62mm" H 4100 2950 50  0001 L CNN
 F 3 "http://www.ti.com/lit/ds/symlink/cd4029b.pdf" H 4100 2850 50  0001 L CNN
 F 4 "CD4029BEE4, 4-stage Decade and Binary Counter Up/Down Counter, Bi-Directional, 3  18 V, 16-Pin PDIP" H 4100 2750 50  0001 L CNN "Description"
@@
 F 0 "U10" H 2450 4100 50  0000 C CNN
 F 1 "CD4029BEE4" H 2650 4000 50  0000 C CNN
-F 2 "DIP794W53P254L1930H508Q16N" H 4100 4000 50  0001 L CNN
+F 2 "Package_DIP:DIP-16_W7.62mm" H 4100 4000 50  0001 L CNN
 F 3 "http://www.ti.com/lit/ds/symlink/cd4029b.pdf" H 4100 3900 50  0001 L CNN
 F 4 "CD4029BEE4, 4-stage Decade and Binary Counter Up/Down Counter, Bi-Directional, 3  18 V, 16-Pin PDIP" H 4100 3800 50  0001 L CNN "Description"
@@
 F 0 "U14" H 4200 6500 50  0000 C CNN
 F 1 "74LS241" H 4300 6400 50  0000 C CNN
-F 2 "" H 4600 5750 50  0001 C CNN
+F 2 "Package_DIP:DIP-20_W7.62mm" H 4600 5750 50  0001 C CNN
 F 3 "http://www.ti.com/lit/ds/symlink/sn74ls241.pdf" H 4600 5750 50  0001 C CNN
 	1    4600 5750
@@
 F 0 "U11" H 2400 5250 50  0000 C CNN
 F 1 "CD4029BEE4" H 2600 5150 50  0000 C CNN
-F 2 "DIP794W53P254L1930H508Q16N" H 4050 5150 50  0001 L CNN
+F 2 "Package_DIP:DIP-16_W7.62mm" H 4050 5150 50  0001 L CNN
 F 3 "http://www.ti.com/lit/ds/symlink/cd4029b.pdf" H 4050 5050 50  0001 L CNN
 F 4 "CD4029BEE4, 4-stage Decade and Binary Counter Up/Down Counter, Bi-Directional, 3  18 V, 16-Pin PDIP" H 4050 4950 50  0001 L CNN "Description"
@@
 F 0 "U12" H 2400 6300 50  0000 C CNN
 F 1 "CD4029BEE4" H 2600 6200 50  0000 C CNN
-F 2 "DIP794W53P254L1930H508Q16N" H 4050 6200 50  0001 L CNN
+F 2 "Package_DIP:DIP-16_W7.62mm" H 4050 6200 50  0001 L CNN
 F 3 "http://www.ti.com/lit/ds/symlink/cd4029b.pdf" H 4050 6100 50  0001 L CNN
 F 4 "CD4029BEE4, 4-stage Decade and Binary Counter Up/Down Counter, Bi-Directional, 3  18 V, 16-Pin PDIP" H 4050 6000 50  0001 L CNN "Description"
@@
 F 0 "U25" H 8450 8450 50  0000 C CNN
 F 1 "74LS241" H 8550 8350 50  0000 C CNN
-F 2 "" H 8850 7700 50  0001 C CNN
+F 2 "Package_DIP:DIP-20_W7.62mm" H 8850 7700 50  0001 C CNN
 F 3 "http://www.ti.com/lit/ds/symlink/sn74ls241.pdf" H 8850 7700 50  0001 C CNN
 	1    8850 7700
@@
 F 0 "U21" H 6650 7200 50  0000 C CNN
 F 1 "CD4029BEE4" H 6850 7100 50  0000 C CNN
-F 2 "DIP794W53P254L1930H508Q16N" H 8300 7100 50  0001 L CNN
+F 2 "Package_DIP:DIP-16_W7.62mm" H 8300 7100 50  0001 L CNN
 F 3 "http://www.ti.com/lit/ds/symlink/cd4029b.pdf" H 8300 7000 50  0001 L CNN
 F 4 "CD4029BEE4, 4-stage Decade and Binary Counter Up/Down Counter, Bi-Directional, 3  18 V, 16-Pin PDIP" H 8300 6900 50  0001 L CNN "Description"
@@
 F 0 "U22" H 6650 8250 50  0000 C CNN
 F 1 "CD4029BEE4" H 6850 8150 50  0000 C CNN
-F 2 "DIP794W53P254L1930H508Q16N" H 8300 8150 50  0001 L CNN
+F 2 "Package_DIP:DIP-16_W7.62mm" H 8300 8150 50  0001 L CNN
 F 3 "http://www.ti.com/lit/ds/symlink/cd4029b.pdf" H 8300 8050 50  0001 L CNN
 F 4 "CD4029BEE4, 4-stage Decade and Binary Counter Up/Down Counter, Bi-Directional, 3  18 V, 16-Pin PDIP" H 8300 7950 50  0001 L CNN "Description"
@@
 F 0 "U26" H 8400 10650 50  0000 C CNN
 F 1 "74LS241" H 8500 10550 50  0000 C CNN
-F 2 "" H 8800 9900 50  0001 C CNN
+F 2 "Package_DIP:DIP-20_W7.62mm" H 8800 9900 50  0001 C CNN
 F 3 "http://www.ti.com/lit/ds/symlink/sn74ls241.pdf" H 8800 9900 50  0001 C CNN
 	1    8800 9900
@@
 F 0 "U23" H 6600 9400 50  0000 C CNN
 F 1 "CD4029BEE4" H 6800 9300 50  0000 C CNN
-F 2 "DIP794W53P254L1930H508Q16N" H 8250 9300 50  0001 L CNN
+F 2 "Package_DIP:DIP-16_W7.62mm" H 8250 9300 50  0001 L CNN
 F 3 "http://www.ti.com/lit/ds/symlink/cd4029b.pdf" H 8250 9200 50  0001 L CNN
 F 4 "CD4029BEE4, 4-stage Decade and Binary Counter Up/Down Counter, Bi-Directional, 3  18 V, 16-Pin PDIP" H 8250 9100 50  0001 L CNN "Description"
@@
 F 0 "U24" H 6600 10450 50  0000 C CNN
 F 1 "CD4029BEE4" H 6800 10350 50  0000 C CNN
-F 2 "DIP794W53P254L1930H508Q16N" H 8250 10350 50  0001 L CNN
+F 2 "Package_DIP:DIP-16_W7.62mm" H 8250 10350 50  0001 L CNN
 F 3 "http://www.ti.com/lit/ds/symlink/cd4029b.pdf" H 8250 10250 50  0001 L CNN
 F 4 "CD4029BEE4, 4-stage Decade and Binary Counter Up/Down Counter, Bi-Directional, 3  18 V, 16-Pin PDIP" H 8250 10150 50  0001 L CNN "Description"
