File: MAX7000CPU-Gen2.sch (KiCad schematic (older format))
At the start: 110 parts, among them J1 Conn_02x05_Odd_Even, J2 Conn_01x08_Male, J4 Conn_01x08_Male, J5 Conn_01x08_Male, J7 Conn_01x05_Male, SW1 SW_Push, SW2 SW_Push, SW3 SW_Push, U1 NE555P, U10 CD4029BEE4, U11 CD4029BEE4, U12 CD4029BEE4, U13 74LS241, U14 74LS241, U15 74LS241, U16 74LS241, U17 74LS574, U18 74LS574, U19 AS6C1008-55PCN, U2 NE555P, U20 74LS574, U21 CD4029BEE4, U22 CD4029BEE4, U23 CD4029BEE4, U24 CD4029BEE4, U25 74LS241, U26 74LS241, U28 74LS574, U29 EPM7128slc84-15n, U3 NE555P, U4 74LS574, U5 74LS574, U6 74LS574, U7 74LS574, U8 74LS574, U9 CD4029BEE4

Commit message: Counter Layout
Parts:
- added R10, R11, R12, R13, R14, R15, R28, R29, R30, R31, R32, R33, R34, R35, R36, R37, R38, R39, R40, R41, R42, R43, R8, R9: 50K, Resistor_THT:R_Axial_DIN0207_L6.3mm_D2.5mm_P7.62mm_Horizontal, symbol MAX7000CPU-Gen2-rescue:R-Device
- renumbered C5 to C1, C14 to C10, C15 to C11, C16 to C12, C17 to C13, C18 to C14, C19 to C15, C20 to C16, C21 to C17, C22 to C18, C23 to C19, C6 to C2, C24 to C20, C25 to C21, C26 to C22, C27 to C23, C28 to C24, C29 to C25, C30 to C26, C31 to C27, C32 to C28, C33 to C29, C34 to C30, C35 to C31, C36 to C32, C37 to C33, C38 to C34, C10 to C35, C9 to C36, C8 to C37, C7 to C38, C1 to C5, C2 to C6, C11 to C7, C12 to C8, C13 to C9, D2 to D1, D11 to D10, D12 to D11, D13 to D12, D14 to D13, D15 to D14, D16 to D15, D17 to D16, D3 to D2, D4 to D3, D5 to D4, D6 to D5, D7 to D6, D8 to D7, D9 to D8, D10 to D9, J4 to J1, J5 to J3, J1 to J4, J7 to J5, R21 to R16, R22 to R17, R12 to R18, R13 to R19, R6 to R2, R14 to R20, R15 to R21, R16 to R22, R17 to R23, R18 to R24, R19 to R25, R23 to R26, R24 to R27, R4 to R3, R5 to R4, R3 to R5, R2 to R6, R20 to R7, SW2 to SW1, SW1 to SW2, U3 to U1, U13 to U10, U15 to U11, U16 to U12, U10 to U13, U11 to U14, U8 to U15, U14 to U16, U12 to U17, U21 to U18, U1 to U2, U25 to U20, U17 to U21, U26 to U24, U18 to U25, U20 to U26, U28 to U27, U24 to U28, U2 to U3, U9 to U7, U29 to U8, U7 to U9
Connections:
- net +5V: now also R15.2, R29.2, R31.2, R32.2, R33.2, R34.2, R35.2, R38.2, R41.2, R42.2, R43.2; no longer U13.10 (UP/DOWN), U13.9 (BINARY/DECADE), U14.10 (UP/DOWN), U14.9 (BINARY/DECADE), U17.10 (UP/DOWN), U17.9 (BINARY/DECADE), U19.30 (CE2), U7.10 (UP/DOWN), U7.9 (BINARY/DECADE)
- net CounterOutControl: now also R15.1, R29.1
- net GND: now also R10.2, R11.2, R12.2, R13.2, R14.2, R28.2, R30.2, R36.1, R37.1, R39.2, R40.2, R8.2, R9.2; no longer U11.1 (OEa), U11.19 (OEb), U12.1 (OEa), U12.19 (OEb), U15.1 (OE), U18.5 (~CARRYIN), U19.2 (A16), U19.22 (~CE), U26.1 (OE), U27.1 (OE), U5.1 (OE), U6.1 (OE), U7.5 (~CARRYIN), U9.1 (OE)
- net MainRegOutputControl: now also R8.1
- net MemOutEnable: now also R33.1
- net MemWriteControl: now also R32.1
- net RAM_Addr_Enable: now also R35.1, R38.1
- net StackOutControl: now also R34.1, R41.1
- new net: R12.1, U9.1 (OE)
- new net: R9.1, U5.1 (OE)
- new net: R10.1, U6.1 (OE)
- new net: R28.1, U15.1 (OE)
- new net: R42.1, U13.10 (UP/DOWN), U14.10 (UP/DOWN), U17.10 (UP/DOWN), U7.10 (UP/DOWN)
- new net: R43.1, U13.9 (BINARY/DECADE), U14.9 (BINARY/DECADE), U17.9 (BINARY/DECADE), U7.9 (BINARY/DECADE)
- new net: R11.1, U7.5 (~CARRYIN)
- new net: R14.1, U12.1 (OEa), U12.19 (OEb)
- new net: R13.1, U11.1 (OEa), U11.19 (OEb)
- new net: R39.1, U26.1 (OE)
- new net: R40.1, U27.1 (OE)
- new net: R30.1, U18.5 (~CARRYIN)
- new net: R37.2, U19.2 (A16)
- new net: R36.2, U19.22 (~CE)
- new net: R31.1, U19.30 (CE2)
Other:
- note removed: "Maybe Pull Chip enables to disable them when controllers arent running\n"
- moved on the sheet: J3

Commit message: PCB component placements
Parts:
- removed R15, R38, R41: 50K, Resistor_THT:R_Axial_DIN0207_L6.3mm_D2.5mm_P7.62mm_Horizontal, symbol MAX7000CPU-Gen2-rescue:R-Device
Other:
- moved on the sheet: R39, R40, U26, U27
